File: analyzer-board/analyzer-board.kicad_pcb (KiCad board)
At the start: 2 copper layers, 90.8 x 90.8 mm, 19 parts, among them J1 Conn_02x20, J2 Conn_01x01, SW1 SW_Push, U1 Teensy4_1_GPIO, U2 74LVC245, U3 74LVC245, U4 74LVC245, U5 74LVC245, U6 74LVC245

Commit message: Fix a PCB error: The wrong footprint was used for the 6mm push button, causing the button input pin on the Teensy to be connected directly to ground.  Fix this problem by using the correct footprint and running a new trace to the correct pad.  Existing boards can be reworked by cutting a trace and using a bodge wire.
Bump schematic and PCB rev to 1.1.
Parts:
- SW1: footprint Button_Switch_THT:SW_TH_Tactile_Omron_B3F-10xx -> Button_Switch_THT:SW_PUSH_6mm
Routing:
- net GND: track 418.7 -> 410.3 mm
