File: analyzer-board/analyzer-board.sch (KiCad schematic (older format))
At the start: 15 parts, among them J1 Conn_02x20, J2 Conn_01x01, SW1 SW_Push, U1 Teensy4_1_GPIO, U2 74LVC245, U3 74LVC245, U4 74LVC245, U5 74LVC245, U6 74LVC245

Commit message: Fix a PCB error: The wrong footprint was used for the 6mm push button, causing the button input pin on the Teensy to be connected directly to ground.  Fix this problem by using the correct footprint and running a new trace to the correct pad.  Existing boards can be reworked by cutting a trace and using a bodge wire.
Bump schematic and PCB rev to 1.1.
Parts:
- SW1: footprint Button_Switch_THT:SW_TH_Tactile_Omron_B3F-10xx -> Button_Switch_THT:SW_PUSH_6mm
Changed lines of the file:
@@
 Sheet 1 1
 Title "TeensyLogicAnalyzer main board"
-Date "2022-04-30"
-Rev "1.0"
+Date "2022-05-21"
+Rev "1.1"
 Comp "Copyright (c) 2022 Jason R. Thorpe.  See LICENSE."
 Comment1 ""
@@
 F 0 "SW1" H 3000 4835 50  0000 C CNN
 F 1 "SW_Push" H 3000 4744 50  0000 C CNN
-F 2 "Button_Switch_THT:SW_TH_Tactile_Omron_B3F-10xx" H 3000 4750 50  0001 C CNN
+F 2 "Button_Switch_THT:SW_PUSH_6mm" H 3000 4750 50  0001 C CNN
 F 3 "~" H 3000 4750 50  0001 C CNN
 	1    3000 4550
@@
 NoConn ~ 11500 500
 $Comp
-L power:GND #PWR?
+L power:GND #PWR0114
 U 1 1 628983B4
 P 8950 4400
-F 0 "#PWR?" H 8950 4150 50  0001 C CNN
+F 0 "#PWR0114" H 8950 4150 50  0001 C CNN
 F 1 "GND" V 8955 4272 50  0000 R CNN
 F 2 "" H 8950 4400 50  0001 C CNN
@@
 $EndComp
 $Comp
-L power:GND #PWR?
+L power:GND #PWR0115
 U 1 1 62898A39
 P 8450 4400
-F 0 "#PWR?" H 8450 4150 50  0001 C CNN
+F 0 "#PWR0115" H 8450 4150 50  0001 C CNN
 F 1 "GND" V 8455 4272 50  0000 R CNN
 F 2 "" H 8450 4400 50  0001 C CNN
